File: yac64pla.kicad_sch (KiCad schematic)
At the start: 3 parts, among them U1 GAL20V8_L, U2 GAL20V8_R, U3 C64_PLA

Commit message: Rename left/right to top/bottom
Parts:
- U1: value GAL20V8_L -> PLD_BOTTOM
- U2: value GAL20V8_R -> PLD_BOTTOM
Changed lines of the file:
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@@
       (effects (font (size 1.27 1.27)) (justify left))
     )
-    (property "Value" "GAL20V8_R" (id 1) (at 131.5594 19.812 0)
+    (property "Value" "PLD_BOTTOM" (id 1) (at 131.5594 19.812 0)
       (effects (font (size 1.27 1.27)) (justify left))
     )
@@
       (effects (font (size 1.27 1.27)) (justify left))
     )
-    (property "Value" "GAL20V8_L" (id 1) (at 57.8994 19.812 0)
+    (property "Value" "PLD_BOTTOM" (id 1) (at 57.8994 19.812 0)
       (effects (font (size 1.27 1.27)) (justify left))
     )
@@
     )
     (path "/e092c7ae-5dc4-42e1-9b43-28f40f25cebf"
-      (reference "U1") (unit 1) (value "GAL20V8_L") (footprint "Package_LCC:PLCC-28")
+      (reference "U1") (unit 1) (value "PLD_TOP") (footprint "Package_LCC:PLCC-28")
     )
     (path "/b0e14891-ade3-41a8-a1ed-ca5b421cb573"
-      (reference "U2") (unit 1) (value "GAL20V8_R") (footprint "Package_LCC:PLCC-28")
+      (reference "U2") (unit 1) (value "PLD_BOTTOM") (footprint "Package_LCC:PLCC-28")
     )
     (path "/851e7b1c-259f-42bc-9440-0054649e3241"
